Commit message: Modify joint limit

File: denso_robot_descriptions/vs087_description/vs087/vs087.urdf.xacro (robot description, xacro)
@@ -127,5 +127,6 @@
 		<origin rpy="0.000000 0.000000 0.000000" xyz="0.000000 0.000000 0.445000" />
 		<axis xyz="-0.000000 1.000000 -0.000000" />
-		<limit effort="1" lower="-1.1836822987" upper="2.54469004941" velocity="3.45575191894877" />
+		<!-- <limit effort="1" lower="-1.1836822987" upper="2.54469004941" velocity="3.45575191894877" /> -->
+		<limit effort="1" lower="-1.1836822987" upper="2.56" velocity="3.45575191894877" />
 		<dynamics damping="0" friction="0" />
 	</joint>
