Commit message: [modify] kinect center position

File: denso_robot_descriptions/vs087_description/vs087_and_robotiq_with_1_kinect/vs087_and_robotiq_with_1_kinect.urdf.xacro (robot description, xacro)
@@ -14,5 +14,6 @@
     <!-- <origin xyz="1.2297 0.1072 0.4985" rpy="-0.0047 0.5886 3.098" />> -->
     <!-- <origin xyz="0.8567 0.0762 0.9535" rpy="-0.0338 0.8795 3.0507" /> -->
-    <origin xyz="0.8834 0.0504 0.9911" rpy="-0.0078 0.6452 -3.1362" />
+    <!-- <origin xyz="0.8834 0.0504 0.9911" rpy="-0.0078 0.6452 -3.1362" /> -->
+    <origin xyz="0.9904 0.1482 0.9801" rpy="0.0151 0.6653 -3.1318" />
     <parent link="world"/>
     <child link="kinect_center_link"/>

Commit message: update

File: denso_robot_descriptions/vs087_description/vs087_and_robotiq_with_1_kinect/vs087_and_robotiq_with_1_kinect.urdf.xacro (robot description, xacro)
@@ -3,6 +3,6 @@
   <!-- <xacro:include filename="$(find denso_robot_descriptions)/vs087_description/vs087/vs087.urdf.xacro"/> -->
   <xacro:include filename="$(find denso_robot_descriptions)/vs087_description/vs087_and_robotiq/vs087_and_robotiq.urdf.xacro"/>
-  <xacro:include filename="$(find kinect_bringup)/urdf/sensor/kinect.urdf.xacro"/>
-  <xacro:include filename="$(find kinect_bringup)/urdf/sensor/kinect.gazebo.xacro"/>
+  <xacro:include filename="$(find denso_robot_description)/kinect_description/kinect.urdf.xacro"/>
+  <xacro:include filename="$(find denso_robot_description)/kinect_description/kinect.gazebo.xacro"/>
   <!-- add Kinect V2 -->
   <!-- kinect_center -->

File: denso_robot_descriptions/vs087_description/vs087_mhand_and_kinect/vs087_mhand_and_kinect.urdf.xacro (robot description, xacro)
@@ -2,7 +2,13 @@
 <robot name="vs087" xmlns:xacro="http://ros.org/wiki/xacro">
   <!-- File Include -->
-  <xacro:include filename="$(find kinect_bringup)/urdf/sensor/kinect.urdf.xacro"/>
-  <xacro:include filename="$(find kinect_bringup)/urdf/sensor/kinect.gazebo.xacro"/>
+    <xacro:include filename="$(find kinect_bringup)/urdf/sensor/kinect.urdf.xacro"/>
+    <xacro:include filename="$(find kinect_bringup)/urdf/sensor/kinect.urdf.xacro"/>
   <xacro:include filename="$(find denso_robot_descriptions)/vs087_description/vs087/vs087.urdf.xacro"/>
+  <xacro:include filename="$(find mhand_description)/robots/mhand.urdf.xacro"/>
+  <joint name="gripper_joint" type="fixed">
+    <origin xyz="0 0 0" rpy="0 0 0"/>
+  <parent link="J6"/>
+  <child link="hand_link"/>
+  </joint>
   <!-- add Kinect V2 -->
   <!-- kinect_center -->
